Commit message: Added namespace for multiagents
need to work on camera and possibly delayed launch

File: description/camera.xacro (robot description, xacro)
@@ -52,5 +52,8 @@
                 </clip>
             </camera>
-            <plugin name="$(arg robot_name)_camera_controller" filename="libgazebo_ros_camera.so">
+            <plugin name="camera_controller" filename="libgazebo_ros_camera.so">
+                <ros>
+                    <namespace>$(arg robot_name)</namespace>
+                </ros>
                 <frame_name>$(arg robot_name)_camera_optical</frame_name> <!-- due to different standards in ros and gazebo -->
             </plugin>

File: description/gazebo_control.xacro (robot description, xacro)
@@ -4,6 +4,6 @@
         <plugin name="$(arg robot_name)_diff_drive" filename="libgazebo_ros_diff_drive.so">
             <!-- Wheel information -->
-            <left_joint>left_front_wheel_joint</left_joint>
-            <right_joint>right_front_wheel_joint</right_joint>
+            <left_joint>$(arg robot_name)_left_front_wheel_joint</left_joint>
+            <right_joint>$(arg robot_name)_right_front_wheel_joint</right_joint>
             <wheel_separation>0.22</wheel_separation>
             <wheel_diameter>0.07</wheel_diameter>
@@ -13,5 +13,5 @@
             <!-- Outputs -->
             <odometry_frame>odom</odometry_frame>
-            <robot_base_frame>base_link</robot_base_frame>
+            <robot_base_frame>$(arg robot_name)_base_link</robot_base_frame>
             <publish_odom>true</publish_odom>
             <publish_odom_tf>true</publish_odom_tf>

File: description/robot_car.urdf.xacro (robot description, xacro)
@@ -1,6 +1,8 @@
 <?xml version="1.0"?>
 <robot xmlns:xacro="http://www.ros.org/wiki/xacro"  name="robot_car">
+    <echo level="error">test test</echo>
     <xacro:arg name="use_ros2_control" default="true" />
     <xacro:arg name="robot_name" default="robot_1"/>
+    <!-- <xacro:property name="robot_name1" value="${robot_name}" /> -->
     <xacro:include filename="car.xacro" />
     <!-- if else statement for controller types -->
@@ -11,4 +13,5 @@
         <xacro:include filename="gazebo_control.xacro" />
     </xacro:unless>
+    <!-- <xacro:include filename="ros2_control.xacro"/> -->
     <!-- <xacro:include filename="lidar.xacro"/> -->
     <xacro:include filename="camera.xacro"/>

File: description/ros2_control.xacro (robot description, xacro)
@@ -6,24 +6,29 @@
         </hardware>
         <joint name="$(arg robot_name)_left_front_wheel_joint">
-            <command_interface name="$(arg robot_name)_velocity">
+            <command_interface name="velocity">
                 <param name="min">-10</param>
                 <param name="max">10</param>
             </command_interface>
-            <state_interface name="$(arg robot_name)_velocity"/>
-            <state_interface name="$(arg robot_name)_position"/>
+            <state_interface name="velocity"/>
+            <state_interface name="position"/>
         </joint>
         <joint name="$(arg robot_name)_right_front_wheel_joint">
-            <command_interface name="$(arg robot_name)_velocity">
+            <command_interface name="velocity">
                 <param name="min">-10</param>
                 <param name="max">10</param>
             </command_interface>
-            <state_interface name="$(arg robot_name)_velocity"/>
-            <state_interface name="$(arg robot_name)_position"/>
+            <state_interface name="velocity"/>
+            <state_interface name="position"/>
         </joint>
     </ros2_control>
     <gazebo>
-        <plugin name="$(arg robot_name)_gazebo_ros2_control" filename="libgazebo_ros2_control.so">
-            <parameters>$(find multi_bear_form)/config/ros2_controller.yaml</parameters>
+        <plugin name="gazebo_ros2_control" filename="libgazebo_ros2_control.so">
+            <ros>
+                <namespace>$(arg robot_name)</namespace>
+            </ros>
+            <parameters>$(find multi_bear_form)/config/$(arg robot_name)_ros2_controller.yaml</parameters>
+            <robot_param_node>/$(arg robot_name)/robot_state_publisher</robot_param_node>
         </plugin>
     </gazebo>
 </robot>
+            <!-- put this below parameters in gazebo pligin <robot_param>robot_1/robot_description</robot_param> -->
